File: MHC_MAIN_REV_2/MHC_MAIN_REV_2.kicad_sch (KiCad schematic)
At the start: 42 parts, among them J1 USB_B_Micro, J2 Conn_ARM_JTAG_SWD_10, J3 BATT, J4 OLED, SW1 RESET, SW2 BOOT, SW3 RotaryEncoder_Switch, SW4 SW_SPDT, SW5 Button_0, U1 MDBT50Q-P1MV2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

Commit message: Updating MHC files
Parts:
- removed J1: USB_B_Micro, Connector_USB:USB_Micro-B_Molex_47346-0001, symbol Connector:USB_B_Micro
- removed R7: 10k, Resistor_SMD:R_0603_1608Metric, symbol Device:R
- removed SW2: BOOT, Button_Switch_SMD:SW_Push_SPST_NO_Alps_SKRK, symbol Switch:SW_Push
- added D5: RED, LED_SMD:LED_0603_1608Metric, symbol Device:LED
- added D6: SK6812MINI, LED_SMD:LED_SK6812MINI_PLCC4_3.5x3.5mm_P1.75mm, symbol LED:SK6812MINI
- added J1: USB_C_Receptacle_USB2.0, Connector_USB:USB_C_Receptacle_G-Switch_GT-USB-7010ASV, symbol Connector:USB_C_Receptacle_USB2.0
- added R10, R11: 5k1, Resistor_SMD:R_0603_1608Metric, symbol Device:R
- added R13: 1k, Resistor_SMD:R_0603_1608Metric, symbol Device:R
- J3: footprint Connector_PinSocket_2.54mm:PinSocket_1x02_P2.54mm_Vertical -> Connector_JST:JST_PH_S2B-PH-SM4-TB_1x02-1MP_P2.00mm_Horizontal
- R1, R2: LCSC C25190 -> (none)
- SW4: footprint Button_Switch_SMD:SW_SPDT_PCM12 -> Connector_PinHeader_2.54mm:PinHeader_1x03_P2.54mm_Vertical
Connections:
- net +3.3V: now also R13.1
- net D+: now also R1.2; no longer R1.1
- net D-: now also R2.2; no longer R2.1
- net GND: now also D5.1 (K), J1.A1 (GND), J1.A12 (GND), J1.B1 (GND), J1.B12 (GND), R10.2, R11.2
- net P0.13: now also D6.3 (DIN)
- net VBUS: now also J1.A4 (VBUS), J1.A9 (VBUS), J1.B4 (VBUS), J1.B9 (VBUS)
- new net: J1.B5 (CC2), R11.1
- new net: J1.A5 (CC1), R10.1
- new net: J1.A6 (D+), J1.B6 (D+), R1.1
- new net: J1.A7 (D-), J1.B7 (D-), R2.1
- new net: D5.2 (A), R13.2
- no-connect marks 31 -> 32
Other:
- moved on the sheet: C4, C7, D1, J3, R3, R4, U2
